Commit message: Initial commit

File: src/robot_description/urdf/assy.urdf (robot description, URDF)
Before this commit: robot myfirst, 0 links, 4 joints
Joints:
- joint base_to_left_wheel: axis 0 0 1 -> 0 1 0; origin xyz=1.1 -1.3 0.0 rpy=1.5708 0 1.5708 -> xyz=-1.3 1.1 0.0 rpy=0 0 0
- joint base_to_right_wheel: axis 0 0 1 -> 0 1 0; origin xyz=-1.1 -1.3 0.0 rpy=1.5708 0 1.5708 -> xyz=-1.3 -1.1 0.0 rpy=0 0 0
- joint base_to_shaft: origin xyz=0 1.3 -0.35 rpy=0 0 0 -> xyz=1.3 0 -0.35 rpy=0 0 0
- joint shaft_to_caster: origin xyz=0 -0.07 -0.15 rpy=1.5708 0 1.5708 -> xyz=-0.07 0 -0.15 rpy=0 0 0

File: src/robot_description/urdf/body.urdf (robot description, URDF)
Before this commit: robot body, 1 links, 0 joints
Links:
- link base_link: mass None -> 5.0; geometry collision box size=4 2 0.5; visual box size=4 2 0.5

File: src/robot_description/urdf/caster.urdf (robot description, URDF)
Before this commit: robot caster, 1 links, 0 joints
Links:
- link caster_link: mass None -> 0.5; geometry collision cylinder length=0.1 radius=0.15; visual cylinder length=0.1 radius=0.15

File: src/robot_description/urdf/wheel_left.urdf (robot description, URDF)
Before this commit: robot wheel, 1 links, 0 joints
Links:
- link left_wheel_link: mass None -> 0.5; geometry collision cylinder length=0.2 radius=0.75; visual cylinder length=0.2 radius=0.75

File: src/robot_description/urdf/wheel_right.urdf (robot description, URDF)
Before this commit: robot wheel, 1 links, 0 joints
Links:
- link right_wheel_link: mass None -> 0.5; geometry collision cylinder length=0.2 radius=0.75; visual cylinder length=0.2 radius=0.75
